File: can.kicad_sch (KiCad schematic)
At the start: 2 parts, among them U2 ISO1042-Q1

Commit message: change power add buzzer
Connections:
- net VDD renamed +3.3V
Changed lines of the file:
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@@
-		)
-	)
-	(hierarchical_label "VDD"
-		(shape input)
-		(at 53.34 105.41 180)
-		(fields_autoplaced yes)
-		(effects
-			(font
-				(size 1.27 1.27)
-				(bold yes)
-			)
-			(justify right)
 		)
 	)
@@
 					(unit 1)
 				)
+			)
+		)
+	)
+	(symbol
+		(lib_id "power:+3.3V")
+		(at 53.34 105.41 0)
+		(unit 1)
+		(exclude_from_sim no)
+		(in_bom yes)
+		(on_board yes)
+		(dnp no)
+		(fields_autoplaced yes)
+		(property "Reference" "#PWR033"
+			(at 53.34 109.22 0)
+			(effects
+				(font
+					(size 1.27 1.27)
+				)
+				(hide yes)
+			)
+		)
+		(property "Value" "+3.3V"
+			(at 53.34 100.33 0)
+			(effects
+				(font
+					(size 1.27 1.27)
+				)
+			)
+		)
+		(property "Footprint" ""
+			(at 53.34 105.41 0)
+			(effects
+				(font
+					(size 1.27 1.27)
+				)
+				(hide yes)
+			)
+		)
+		(property "Datasheet" ""
+			(at 53.34 105.41 0)
+			(effects
+				(font
+					(size 1.27 1.27)
+				)
+				(hide yes)
+			)
+		)
+		(property "Description" "Power symbol creates a global label with name \"+3.3V\""
+			(at 53.34 105.41 0)
+			(effects
+				(font
+					(size 1.27 1.27)
+				)
+				(hide yes)
+			)
+		)
+		(pin "1"
+		)
+		(instances
+			(project ""
+				(path "/8d063f79-9282-4820-bcf4-1ff3c006cf08/73909d3a-f2e9-43a1-adfe-e0aaff309cf7"
+					(reference "#PWR033")
+					(unit 1)
+				)

Commit message: smaller caps remove ringing resistors
Parts:
- R1: value 120 -> 120R
Changed lines of the file:
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@@
 			)
 		)
-		(property "Value" "120"
+		(property "Value" "120R"
 			(at 182.88 125.73 90)
 			(effects
@@
 			)
 		)
-		(property "Datasheet" "~"
+		(property "Datasheet" "https://wmsc.lcsc.com/wmsc/upload/file/pdf/v2/lcsc/2206010216_UNI-ROYAL-Uniroyal-Elec-0805W8F1200T5E_C17437.pdf"
 			(at 182.88 125.73 0)
 			(effects

Commit message: pre-quilter after cap size issue
Parts:
- U2: footprint Package_SO:SOIC-8_3.9x4.9mm_P1.27mm -> Package_SO:SOIC-8_7.5x5.85mm_P1.27mm
Changed lines of the file:
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@@
 			)
 		)
-		(property "Footprint" "Package_SO:SOIC-8_3.9x4.9mm_P1.27mm"
+		(property "Footprint" "Package_SO:SOIC-8_7.5x5.85mm_P1.27mm"
 			(at 139.7 134.62 0)
 			(effects

Commit message: SENT TO jlcpcb
Parts:
- U2: JLCPCB Rotation Offset (none) -> 90
Changed lines of the file:
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@@
+			)
+		)
+		(property "JLCPCB Rotation Offset" "90"
+			(at 139.7 124.46 0)
+			(effects
+				(font
+					(size 1.27 1.27)
+				)
+				(hide yes)
 			)
 		)
