File: can.kicad_sch (KiCad schematic)
At the start: 2 parts, among them U2 ISO1042-Q1

Commit message: version 2 initial
Parts:
- added C22, C25: 100nF, Capacitor_SMD:C_0603_1608Metric, symbol Device:C
- added C24: 10uF, Capacitor_SMD:C_0805_2012Metric, symbol Device:C
- added J3: JST GH, dnt:JST_GH_BM06B-GHS-TBT_1x06-1MP_P1.25mm_Vertical, symbol PCM_SL_Connectors:JST_06
- added J6: Screw_Terminal_01x06, TerminalBlock_Phoenix:TerminalBlock_Phoenix_PT-1,5-6-3.5-H_1x06_P3.50mm_Horizontal, symbol Connector:Screw_Terminal_01x06
- added JP2: SolderJumper_2_Bridged, Jumper:SolderJumper-2_P1.3mm_Open_TrianglePad1.0x1.5mm, symbol Jumper:SolderJumper_2_Bridged
Connections:
- net +3.3V: now also C22.1
- net +5V_ISO: now also C24.1, C25.1
- net GND: now also C22.2, J3.2, J3.3, J6.2 (Pin_2), J6.3 (Pin_3)
- net GND_ISO: now also C24.2, C25.2, J3.6, J6.6 (Pin_6)
- net CAN_H: no longer names the net of R1.2
- net CAN_H: now also JP2.1 (A); no longer U2.7 (CANH)
- net CAN_L: no longer names the net of R1.1, U2.6 (CANL)
- net CAN_L: now also J3.5, J6.5 (Pin_5)
- new net: J3.4, J6.4 (Pin_4), JP2.2 (B), U2.7 (CANH)
- new net VBATT: J3.1, J6.1 (Pin_1)
Other:
- note added: "Near VCC1"
- note added: "Near VCC2"
- moved on the sheet: R1, U2

Commit message: version 2 initial- fixes
Parts:
- JP2: now not fitted
Connections:
- net CAN_L: now reaches J3.5, J6.5 (Pin_5), R1.1, U2.6 (CANL)
- net CAN_H: now reaches J3.4, J6.4 (Pin_4), JP2.2 (B), U2.7 (CANH)
Changed lines of the file:
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@@
+		)
+	)
+	(label "CAN_H"
+		(at 247.65 85.09 180)
+		(effects
+			(font
+				(size 1.27 1.27)
+			)
+			(justify right bottom)
+		)
+	)
+	(label "GND_ISO"
+		(at 247.65 80.01 180)
+		(effects
+			(font
+				(size 1.27 1.27)
+			)
+			(justify right bottom)
+		)
+	)
+	(label "CAN_L"
+		(at 247.65 82.55 180)
+		(effects
+			(font
+				(size 1.27 1.27)
+			)
+			(justify right bottom)
 		)
 	)
@@
 		(in_bom no)
 		(on_board yes)
-		(dnp no)
+		(dnp yes)
 		(fields_autoplaced yes)
 		(property "Reference" "JP2"

Commit message: SENT TO jlcpcb
Parts:
- C24: footprint Capacitor_SMD:C_0805_2012Metric -> Capacitor_SMD:C_0603_1608Metric
- J3: LCSC (none) -> C189892
- J6: LCSC (none) -> C5290323
Connections:
- net +3.3V renamed +3.3VP
Changed lines of the file:
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@@
 	(label "CAN_H"
 		(at 247.65 85.09 180)
+		(fields_autoplaced yes)
 		(effects
 			(font
@@
 	(label "GND_ISO"
 		(at 247.65 80.01 180)
+		(fields_autoplaced yes)
 		(effects
 			(font
@@
 	(label "CAN_L"
 		(at 247.65 82.55 180)
+		(fields_autoplaced yes)
 		(effects
 			(font
@@
 	)
 	(symbol
-		(lib_id "power:+3.3V")
-		(at 43.18 90.17 0)
-		(unit 1)
-		(exclude_from_sim no)
-		(in_bom yes)
-		(on_board yes)
-		(dnp no)
-		(fields_autoplaced yes)
-		(property "Reference" "#PWR033"
-			(at 43.18 93.98 0)
-			(effects
-				(font
-					(size 1.27 1.27)
-				)
-				(hide yes)
-			)
-		)
-		(property "Value" "+3.3V"
-			(at 43.18 85.09 0)
-			(effects
-				(font
-					(size 1.27 1.27)
-				)
-			)
-		)
-		(property "Footprint" ""
-			(at 43.18 90.17 0)
-			(effects
-				(font
-					(size 1.27 1.27)
-				)
-				(hide yes)
-			)
-		)
-		(property "Datasheet" ""
-			(at 43.18 90.17 0)
-			(effects
-				(font
-					(size 1.27 1.27)
-				)
-				(hide yes)
-			)
-		)
-		(property "Description" "Power symbol creates a global label with name \"+3.3V\""
-			(at 43.18 90.17 0)
-			(effects
-				(font
-					(size 1.27 1.27)
-				)
-				(hide yes)
-			)
-		)
-		(pin "1"
-		)
-		(instances
-			(project "l8-kicad"
-				(path "/8d063f79-9282-4820-bcf4-1ff3c006cf08/73909d3a-f2e9-43a1-adfe-e0aaff309cf7"
-					(reference "#PWR033")
-					(unit 1)
-				)
-			)
-		)
-	)
-	(symbol
 		(lib_id "Device:C")
 		(at 118.11 114.3 0)
@@
 			)
 		)
-		(property "Footprint" "Capacitor_SMD:C_0805_2012Metric"
+		(property "Footprint" "Capacitor_SMD:C_0603_1608Metric"
 			(at 119.0752 118.11 0)
 			(effects
@@
 				(path "/8d063f79-9282-4820-bcf4-1ff3c006cf08/73909d3a-f2e9-43a1-adfe-e0aaff309cf7"
 					(reference "C24")
+					(unit 1)
+				)
+			)
+		)
+	)
+	(symbol
+		(lib_id "power:+3.3VP")
+		(at 43.18 90.17 0)
+		(unit 1)
+		(exclude_from_sim no)
+		(in_bom yes)
+		(on_board yes)
+		(dnp no)
+		(fields_autoplaced yes)
+		(property "Reference" "#PWR026"
+			(at 46.99 91.44 0)
+			(effects
+				(font
+					(size 1.27 1.27)
+				)
+				(hide yes)
+			)
+		)
+		(property "Value" "+3.3VP"
+			(at 43.18 85.09 0)
+			(effects
+				(font
+					(size 1.27 1.27)
+				)
+			)
+		)
+		(property "Footprint" ""
+			(at 43.18 90.17 0)
+			(effects
+				(font
+					(size 1.27 1.27)
+				)
+				(hide yes)
+			)
+		)
+		(property "Datasheet" ""
+			(at 43.18 90.17 0)
+			(effects
+				(font
+					(size 1.27 1.27)
+				)
+				(hide yes)
+			)
+		)
+		(property "Description" "Power symbol creates a global label with name \"+3.3VP\""
+			(at 43.18 90.17 0)
+			(effects
+				(font
+					(size 1.27 1.27)
+				)
+				(hide yes)
+			)
+		)
+		(pin "1"
+		)
+		(instances
+			(project ""
+				(path "/8d063f79-9282-4820-bcf4-1ff3c006cf08/73909d3a-f2e9-43a1-adfe-e0aaff309cf7"
+					(reference "#PWR026")
 					(unit 1)
 				)
@@
 			)
 		)
-		(property "Datasheet" "~"
+		(property "Datasheet" "https://wmsc.lcsc.com/wmsc/upload/file/pdf/v2/lcsc/2304140030_JST-BM06B-GHS-TBT-LF-SN_C189892.pdf"
 			(at 251.46 97.79 0)
 			(effects
@@
 		)
 		(property "Silkscreen" ""
+			(at 251.46 86.36 0)
+			(effects
+				(font
+					(size 1.27 1.27)
+				)
+				(hide yes)
+			)
+		)
+		(property "LCSC" "C189892"
 			(at 251.46 86.36 0)
 			(effects
@@
 			(at 251.46 111.76 0)
 			(effects
+				(font
+					(size 1.27 1.27)
+				)
+				(hide yes)
+			)
+		)
+		(property "LCSC" "C5290323"
+			(at 251.46 111.76 0)
+			(effects

Commit message: update to version 9 on selwyn
Other:
- title: (none) -> l8
