File: l8-kicad.kicad_pcb (KiCad board)
At the start: 2 copper layers, 55.5 x 89.5 mm, 120 parts, among them J1 USB_B_Mini, J2 LCD 3.2" 240x320 Conn_01x14_P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, J3 Screw_Terminal_01x06, J4 Conn_ST_STDC14, J7 TC2030 - TAG Connect, Q1 SI2301CDS-T1-GE3, Q4 SI2301CDS-T1-GE3, Q5 SI2301CDS-T1-GE3, SW1 SW_Push, SW2 SW_Push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

Commit message: pre JLCPCB try 1
Routing:
- net +5V: track 127.7 -> 130.0 mm
- net +3.3V: track 642.5 -> 641.2 mm
- net /MCU/USART2_RX: track 29.5 -> 28.9 mm
- net Net-(U3-VDDA): track 37.8 -> 37.2 mm
- net Net-(D12-A): track 22.8 -> 22.2 mm
- net /MCU/PC14: track 16.8 -> 17.4 mm
- net /SPI1_CS2: track 47.7 -> 47.2 mm
- net /MCU/PD8: track 23.7 -> 23.2 mm

Commit message: change to 2.2k for 12v LED
Parts:
- R4: value 100R -> 2.2K
Changed lines of the file:
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@@
 		(sheetname "usb")
 		(sheetfile "usb.kicad_sch")
-		(attr through_hole exclude_from_bom)
+		(attr through_hole)
 		(fp_line
 			(start 3.9 -2.025)
@@
 			)
 		)
-		(property "Value" "100R"
+		(property "Value" "2.2K"
 			(at 0 1.43 90)
 			(layer "F.Fab")
@@
 			)
 		)
-		(property "LCSC" "C22775"
+		(property "LCSC" "C4190"
 			(at 0 0 90)
 			(unlocked yes)
@@
 			(at 0 0 -90)
 			(unlocked yes)
+			(layer "F.Fab")
+			(hide yes)
+			(effects
+				(font
+					(size 1 1)
+					(thickness 0.15)
+				)
+			)
+		)
+		(property "LCSC" "C C2992393"
+			(at 0 0 -90)
+			(unlocked yes)

Commit message: version 2 changes
Parts:
- removed PS1: D36V6F5, Connector_PinHeader_2.54mm:PinHeader_1x04_P2.54mm_Vertical
- removed TP10: PC8, dnt:TestPoint_Pad_D1.0mm FP .6R
- removed TP11: PC9, dnt:TestPoint_Pad_D1.0mm FP .6R
- removed TP12: PC13, dnt:TestPoint_Pad_D1.0mm FP .6R
- removed TP13: PC14, dnt:TestPoint_Pad_D1.0mm FP .6R
- removed TP14: PC15, dnt:TestPoint_Pad_D1.0mm FP .6R
- removed TP15: PC0, dnt:TestPoint_Pad_D1.0mm FP .6R
- removed TP22: PB8, dnt:TestPoint_Pad_D1.0mm FP .6R
- removed TP24: PB10, dnt:TestPoint_Pad_D1.0mm FP .6R
- removed TP25: PB11, dnt:TestPoint_Pad_D1.0mm FP .6R
- removed TP26: PB12, dnt:TestPoint_Pad_D1.0mm FP .6R
- removed TP27: PD6, dnt:TestPoint_Pad_D1.0mm FP .6R
- removed TP28: PD7, dnt:TestPoint_Pad_D1.0mm FP .6R
- removed TP29: PD8, dnt:TestPoint_Pad_D1.0mm FP .6R
- removed TP30: PD9, dnt:TestPoint_Pad_D1.0mm FP .6R
- removed TP31: PE8, dnt:TestPoint_Pad_D1.0mm FP .6R
- removed TP32: PE7, dnt:TestPoint_Pad_D1.0mm FP .6R
- removed TP33: PE0, dnt:TestPoint_Pad_D1.0mm FP .6R
- removed TP34: PE1, dnt:TestPoint_Pad_D1.0mm FP .6R
- removed TP35: PE9, dnt:TestPoint_Pad_D1.0mm FP .6R
- removed TP36: PE10, dnt:TestPoint_Pad_D1.0mm FP .6R
- removed TP37: PE11, dnt:TestPoint_Pad_D1.0mm FP .6R
- removed TP38: PE12, dnt:TestPoint_Pad_D1.0mm FP .6R
- removed TP39: PD10, dnt:TestPoint_Pad_D1.0mm FP .6R
- removed TP40: PD11, dnt:TestPoint_Pad_D1.0mm FP .6R
- removed TP6: 5V ISO, dnt:TestPoint_Pad_D1.0mm FP .6R
- removed TP8: PC6, dnt:TestPoint_Pad_D1.0mm FP .6R
- removed TP9: PC7, dnt:TestPoint_Pad_D1.0mm FP .6R
- added C3: 10uF, Capacitor_SMD:C_0805_2012Metric, F.Cu at (152.2, 115.5)
- added D7: SS14, dnt:D_SMA - polarity, F.Cu at (150.0, 126.0)
- added D8: LED-RED, LED_SMD:LED_0603_1608Metric, F.Cu at (153.2, 111.8)
- added F1: Fuse, Fuse:Fuse_0805_2012Metric, F.Cu at (146.5, 156.0)
- added F2: Fuse, Fuse:Fuse_0805_2012Metric, F.Cu at (143.4, 120.0)
- added F3: Fuse, Fuse:Fuse_0805_2012Metric, F.Cu at (146.5, 107.2)
- added L1: 3.3uH, Inductor_SMD:L_Sunlord_SWPA4030S, F.Cu at (142.8, 126.2)
- added R20: 2.2K, Resistor_SMD:R_0603_1608Metric, F.Cu at (148.6, 111.8)
- added R6: 100R, Resistor_SMD:R_0603_1608Metric, F.Cu at (145.2, 175.3)
- added U6: LMR14006, Package_TO_SOT_SMD:SOT-23-6, F.Cu at (148.9, 119.2)
- D2: footprint Diode_SMD:D_SMA -> dnt:D_SMA - polarity
- J4: footprint dnt:CON14_2X7_DUK_FTSH_SAI -> dnt:SAMTEC_FTSH-107-01-F-DV-K-Fix
- J7: value TC2030 - TAG Connect -> TC2070 - TAG Connect; footprint Connector:Tag-Connect_TC2030-IDC-NL_2x03_P1.27mm_Vertical -> Connector:Tag-Connect_TC2070-IDC-FP_2x07_P1.27mm_Vertical
- U4: footprint Package_DIP:DIP-24_W15.24mm_Socket -> dnt:DIP-24_W15.24mm_Socket- nox
- moved TP2 21.5 mm to (154.0, 131.0), turned to 0 degrees
- moved R1 13.6 mm to (144.8, 147.2), turned to -90 degrees
- moved TP1 12.8 mm to (153.2, 109.5)
- moved J3 11.3 mm to (150.3, 151.5)
- moved R2 10.8 mm to (133.0, 118.8)
- moved U1 10.0 mm to (140.0, 132.9)
- moved D2 9.35 mm to (151.2, 156.0), turned to 180 degrees
- moved J7 8.31 mm to (150.7, 174.6)
- moved TP20 8.13 mm to (135.5, 161.2)
- moved U22 8.10 mm to (142.5, 111.5)
- moved C5 7.81 mm to (142.5, 105.0)
- moved R4 7.63 mm to (144.2, 155.8)
- moved C4 7.62 mm to (142.5, 109.2)
- moved C7 7.62 mm to (142.7, 107.2)
- moved D3 7.29 mm to (151.8, 163.3)
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Connections:
- net /SPI3_CS renamed /SPI4_CS_2
- net /SPI4_CS renamed /SPI4_CS_1
- C4 pad 1: +3.3V -> Net-(U22-OUT)
- C5 pad 2: +3.3V -> Net-(U22-OUT)
- C7 pad 1: +3.3V -> Net-(U22-OUT)
- D2 pad 2: /VBATT -> Net-(D2-A)
- J2 pad 6: /SPI3_SDO -> /SPI4_SDO
- J2 pad 7: /SPI3_SCK -> /SPI4_SCK
- J2 pad 9: /SPI3_SDI -> /SPI4_SDI
- J3 pad 4: /CAN_L -> /CAN_H
- J3 pad 5: /CAN_H -> /CAN_L
- J7 pad 1: +3.3V -> unconnected-(J7-NC-Pad1)
- J7 pad 2: /MCU/SYS_JTMS-SWDIO -> unconnected-(J7-NC-Pad2)
- J7 pad 3: /MCU/NRST -> +3.3V
- J7 pad 4: /MCU/SYS_JTCK-SWCLK -> /MCU/SYS_JTMS-SWDIO
- J7 pad 6: /MCU/SYS_JTDO-SWO -> /MCU/SYS_JTCK-SWCLK
- R27 pad 2: /SPI3_SCK -> /MCU/SPI3_SCK
- R28 pad 2: /SPI3_SDI -> /MCU/SPI3_SDI
- R29 pad 2: /SPI3_SDO -> /MCU/SPI3_SDO
- U22 pad 1: +3.3V -> Net-(U22-OUT)
- U22 pad 2: +3.3V -> Net-(U22-OUT)
Routing:
- net +3.3V: track 641.2 -> 558.0 mm, vias 30 -> 17
- net /SPI3_SDO: track 63.6 -> 0.00 mm, vias 1 -> 0
- net Net-(D1-A): track 48.6 -> 0.00 mm
- net /SPI4_CS_2: track 126.1 -> 90.1 mm, vias 3 -> 4
- net /MCU/USART2_TX: track 149.3 -> 113.9 mm, vias 4 -> 5
- net /MCU/PC0: track 26.9 -> 0.00 mm, vias 4 -> 0
- net /MCU/PD7: track 26.5 -> 0.00 mm, vias 2 -> 0
- net /MCU/PD9: track 26.4 -> 0.00 mm, vias 2 -> 0
- net /MCU/PE7: track 26.2 -> 0.00 mm
- net /MCU/PD10: track 25.9 -> 0.00 mm, vias 2 -> 0
- net /MCU/SYS_JTMS-SWDIO: track 64.0 -> 38.8 mm
- net /MCU/PE11: track 24.7 -> 0.00 mm, vias 2 -> 0
- net /MCU/PD8: track 23.2 -> 0.00 mm
- net /MCU/PC13: track 21.9 -> 0.00 mm, vias 2 -> 0
- net /MCU/PE12: track 20.6 -> 0.00 mm, vias 2 -> 0
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- added copper zone on B.Cu, net +5V
- added copper zone on F.Cu, net +5V
- removed copper zone on B.Cu, net GND
- removed copper zone on F.Cu, net GND
Other:
- board text added: "L8 - XXXXXXXX062024"
- board text added: "RESET"
- board text removed: "12V"
- board text removed: "GND"
- board text removed: "L8 - 07062024"
- board text removed: "NRST"

Commit message: x
Parts:
- removed Q4, Q5: SI2301CDS-T1-GE3, Package_TO_SOT_SMD:SOT-23
- removed R27, R28, R29: 22R, Resistor_SMD:R_0603_1608Metric
- added Q2: AO3400A, Package_TO_SOT_SMD:SOT-23, F.Cu at (113.9, 115.0)
- added Q3: AO3400A, Package_TO_SOT_SMD:SOT-23, F.Cu at (106.7, 139.3)
- added R18: 2.2K, Resistor_SMD:R_0603_1608Metric, F.Cu at (148.8, 115.2)
- added R19: 2.2K, Resistor_SMD:R_0603_1608Metric, F.Cu at (145.3, 114.0)
- D1, D11, D4, D5, D6, D8: footprint LED_SMD:LED_0603_1608Metric -> dnt:LED_0603_1608Metric - polarity
- D12: footprint Diode_SMD:D_SOD-123 -> dnt:D_SOD-123-polarity
- FB1: value ~ -> 4.7uH
- Q1: value SI2301CDS-T1-GE3 -> AO3400A
- moved TP2 9.86 mm to (144.2, 129.5)
- moved R14 5.08 mm to (111.0, 114.8), turned to 90 degrees
- moved R3 4.06 mm to (109.2, 114.8)
- moved R32 3.48 mm to (102.0, 139.2)
- moved R33 1.85 mm to (103.8, 139.2), turned to 90 degrees
- moved Q1 1.40 mm to (132.9, 114.2)
- moved TP1 0.90 mm to (154.0, 110.0)
Connections:
- Q1 pad 2: Net-(Q1-D) -> GND
- Q1 pad 3: GND -> Net-(Q1-D)
- U6 pad 3: unconnected-(U6-FB-Pad3) -> Net-(U6-FB)
Routing:
- net /MCU/SPI3_SCK_*: track 70.5 -> 0.00 mm, vias 4 -> 0
- net /MCU/SPI3_SDI_*: track 64.6 -> 0.00 mm, vias 2 -> 0
- net /MCU/USART2_TX: track 113.9 -> 60.4 mm, vias 5 -> 3
- net /MCU/SPI3_SDO_*: track 17.6 -> 0.00 mm
- net +5V: track 126.6 -> 109.3 mm, vias 126 -> 8
- net Net-(Q2-G): track 11.8 -> 3.42 mm
- net Net-(Q1-G): track 0.00 -> 5.60 mm, vias 1 -> 0
- net /LCD_ON: track 51.9 -> 56.1 mm
- net /MCU/BEEPER: track 39.2 -> 42.7 mm
- net Net-(Q3-G): track 7.07 -> 3.75 mm
- net Net-(Q1-D): track 65.4 -> 62.4 mm
- net Net-(BZ1--): track 17.9 -> 15.1 mm
- net /LCD_RESET: track 76.9 -> 74.2 mm, vias 6 -> 2
- net +3.3V: track 558.0 -> 555.4 mm
- net Net-(J2-GND): track 16.4 -> 14.6 mm
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- added copper zone on B.Cu, net GND
- added copper zone on F.Cu, net GND
- removed copper zone on B.Cu, net +5V
- removed copper zone on F.Cu, net +5V

Commit message: 5v buck
Parts:
- added C18: C, Capacitor_SMD:C_0805_2012Metric, F.Cu at (148.6, 121.5)
- added C19: C, Capacitor_SMD:C_0805_2012Metric, F.Cu at (144.7, 113.8)
- added C21: 10uF, Capacitor_SMD:C_0805_2012Metric, F.Cu at (144.3, 108.3)
- added D9: LED-RED, dnt:LED_0603_1608Metric - polarity, F.Cu at (102.4, 110.7)
- added J6: JST GH, dnt:JST_GH_BM06B-GHS-TBT_1x06-1MP_P1.25mm_Vertical, F.Cu at (152.2, 130.1)
- added R21: 2.2K, Resistor_SMD:R_0603_1608Metric, F.Cu at (106.3, 110.5)
- R18: value 2.2K -> 1.02k
- R19: value 2.2K -> 5.62
- U1: footprint dnt:B0505S-1WR2_MNS -> dnt:0505_Isolated_SMD
- moved D8 51.0 mm to (102.3, 108.8), turned to 180 degrees
- moved TP1 47.1 mm to (107.0, 107.0)
- moved R20 42.4 mm to (106.2, 108.8), turned to 180 degrees
- moved TP2 14.4 mm to (130.0, 131.8)
- moved D7 14.2 mm to (148.1, 112.0), turned to 90 degrees
- moved D2 11.2 mm to (140.5, 159.0)
- moved L1 8.87 mm to (146.0, 118.0), turned to 180 degrees
- moved R19 7.99 mm to (145.8, 122.0), turned to -90 degrees
- moved R18 7.17 mm to (151.2, 122.0), turned to -90 degrees
- moved R4 5.18 mm to (144.5, 150.6), turned to -90 degrees
- moved J3 4.46 mm to (150.0, 155.9)
- moved F1 3.78 mm to (146.0, 159.8), turned to 180 degrees
- moved D1 3.44 mm to (144.5, 154.0), turned to -90 degrees
- moved U1 3.32 mm to (139.8, 136.2), turned to 0 degrees
- moved F2 3.31 mm to (142.2, 123.0), turned to -90 degrees
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Connections:
- U1 pad 4: /+5V_ISO -> /GND_ISO
- U6 pad 1: unconnected-(U6-CB-Pad1) -> Net-(U6-CB)
Routing:
- net +5V: track 109.3 -> 185.9 mm, vias 8 -> 10
- net /VBATT: track 0.00 -> 38.7 mm
- net Net-(BZ1--): track 15.1 -> 35.4 mm
- net Net-(D1-A): track 0.00 -> 18.8 mm
- net /CAN_H: track 17.0 -> 31.5 mm
- net /+5V_ISO: track 0.00 -> 10.0 mm, vias 0 -> 2
- net Net-(U6-FB): track 0.00 -> 9.44 mm
- net +3.3V: track 555.4 -> 564.2 mm, vias 17 -> 18
- net Net-(D2-A): track 0.00 -> 8.49 mm
- net /GND_ISO: track 17.4 -> 25.3 mm
- net /CAN_L: track 18.6 -> 25.9 mm
- net Net-(C19-Pad1): track 0.00 -> 6.65 mm
- net GND: track 12.1 -> 16.9 mm, vias 121 -> 135
- net Net-(D7-K): track 0.00 -> 3.63 mm
- net Net-(U6-CB): track 0.00 -> 2.15 mm
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
Commit message: version 2 initial
Parts:
- removed C29: 10nF, Capacitor_SMD:C_0603_1608Metric
- removed D7: SS14, dnt:D_SMA - polarity
- removed TP16: PA0, dnt:TestPoint_Pad_D1.0mm FP .6R
- added C22: 100nF, Capacitor_SMD:C_0603_1608Metric, F.Cu at (135.4, 154.2)
- added C24: 10uF, Capacitor_SMD:C_0805_2012Metric, F.Cu at (135.3, 148.3)
- added C25: 100nF, Capacitor_SMD:C_0603_1608Metric, F.Cu at (135.6, 144.8)
- added C26: 10uF, Capacitor_SMD:C_0805_2012Metric, F.Cu at (115.3, 171.4)
- added D13: ~, Diode_SMD:D_MicroSMP_AK, F.Cu at (149.5, 111.3)
- added J10: Conn_01x04_Pin, Connector_PinSocket_2.54mm:PinSocket_1x04_P2.54mm_Vertical, F.Cu at (123.6, 187.4)
- added JP2: SolderJumper_2_Bridged, Jumper:SolderJumper-2_P1.3mm_Open_TrianglePad1.0x1.5mm, F.Cu at (145.1, 144.3)
- added JP3: SolderJumper_2_Open, Jumper:SolderJumper-2_P1.3mm_Open_TrianglePad1.0x1.5mm, F.Cu at (102.5, 117.5)
- added JP4: SolderJumper_2_Bridged, Jumper:SolderJumper-2_P1.3mm_Open_TrianglePad1.0x1.5mm, F.Cu at (102.5, 114.8)
- added U7: SN74LVC1G14DRL, Package_TO_SOT_SMD:SOT-553, F.Cu at (126.2, 136.2)
- J3: value Screw_Terminal_01x06 -> JST GH; footprint TerminalBlock_Phoenix:TerminalBlock_Phoenix_PT-1,5-6-3.5-H_1x06_P3.50mm_Horizontal -> dnt:JST_GH_BM06B-GHS-TBT_1x06-1MP_P1.25mm_Vertical
- J6: value JST GH -> Screw_Terminal_01x06; footprint dnt:JST_GH_BM06B-GHS-TBT_1x06-1MP_P1.25mm_Vertical -> TerminalBlock_Phoenix:TerminalBlock_Phoenix_PT-1,5-6-3.5-H_1x06_P3.50mm_Horizontal
- moved J6 12.1 mm to (150.4, 142.1), turned to 90 degrees
- moved TP18 10.4 mm to (116.8, 155.2)
- moved R19 6.04 mm to (151.5, 119.8)
- moved R12 5.87 mm to (108.0, 125.8)
- moved J3 5.60 mm to (150.6, 150.4), turned to -90 degrees
- moved F2 5.34 mm to (146.5, 120.0)
- moved C23 4.71 mm to (111.0, 158.2), turned to 90 degrees
- moved TP19 4.50 mm to (131.7, 175.8)
- moved C16 4.18 mm to (133.8, 171.9), turned to 90 degrees
- moved C19 3.71 mm to (147.4, 111.4)
- moved R16 3.32 mm to (133.2, 183.4), turned to 90 degrees
- moved L1 2.89 mm to (147.9, 115.9)
- moved U6 2.89 mm to (152.2, 116.1)
- moved R18 2.89 mm to (153.2, 119.8)
- moved C3 2.86 mm to (151.7, 111.5)
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Connections:
- net /CAN_L renamed Net-(J6-Pin_5)
- C10 pad 2: Net-(Q1-D) -> GND
- C18 pad 2: Net-(D7-K) -> Net-(D13-K)
- C19 pad 1: Net-(C19-Pad1) -> Net-(D13-K)
- C2 pad 2: Net-(Q1-D) -> GND
- F2 pad 1: Net-(C19-Pad1) -> Net-(D13-K)
- J2 pad 14: /SPI4_IRQ -> Net-(J2-T_IRQ)
- J3 pad 4: /CAN_H -> Net-(J6-Pin_4)
- J4 pad 10: /MCU/SYS_JTDI -> unconnected-(J4-JTDI/NC-Pad10)
- J6 pad 4: /CAN_H -> Net-(J6-Pin_4)
- J7 pad 10: /MCU/SYS_JTDI -> unconnected-(J7-JTDI/NC-Pad10)
- L1 pad 1: Net-(D7-K) -> Net-(D13-K)
- L1 pad 2: Net-(C19-Pad1) -> Net-(D13-K)
- Q2 pad 3: Net-(J2-GND) -> Net-(JP3-A)
- R1 pad 2: /CAN_H -> Net-(JP2-A)
- R10 pad 1: Net-(Q1-D) -> GND
- R11 pad 1: Net-(Q1-D) -> GND
- R12 pad 1: Net-(Q1-D) -> GND
- R19 pad 1: Net-(C19-Pad1) -> Net-(D13-K)
- R9 pad 1: Net-(Q1-D) -> GND
- U2 pad 7: /CAN_H -> Net-(J6-Pin_4)
- U3 pad 17: /SPI2_SDO -> /SPI2_SDI
- U3 pad 18: /SPI2_SDI -> /SPI2_SDO
- U3 pad 23: /MCU/PA0 -> /SYS_WAKEUP
- U3 pad 3: /SPI4_IRQ -> /MCU/SPI4_IRQ
- U3 pad 77: /MCU/SYS_JTDI -> /SPI3_CS
- U3 pad 78: /MCU/SPI3_SCK_* -> /SPI3_SCK
- U3 pad 79: /MCU/SPI3_SDI_* -> /SPI3_SDI
- U3 pad 80: /MCU/SPI3_SDO_* -> /SPI3_SDO
- U6 pad 4: unconnected-(U6-~{SHDN}-Pad4) -> Net-(D1-A)
- U6 pad 6: Net-(D7-K) -> Net-(D13-K)
Routing:
- net +3.3V: track 564.2 -> 455.8 mm, vias 18 -> 16
- net /SPI4_IRQ: track 62.9 -> 0.00 mm
- net Net-(J2-T_IRQ): track 0.00 -> 52.3 mm, vias 0 -> 2
- net Net-(D1-A): track 18.8 -> 62.8 mm
- net /GND_ISO: track 25.3 -> 67.7 mm
- net /MCU/SYS_JTDI: track 35.3 -> 0.00 mm
- net /CAN_H: track 31.5 -> 0.00 mm
- net Net-(J6-Pin_4): track 0.00 -> 30.5 mm
- net /SYS_WAKEUP: track 0.00 -> 26.2 mm, vias 0 -> 4
- net /SPI3_SDI: track 0.00 -> 25.0 mm, vias 0 -> 1
- net /SPI3_CS: track 0.00 -> 24.6 mm, vias 0 -> 1
- net /SPI3_SDO: track 0.00 -> 23.7 mm, vias 0 -> 1
- net /SPI3_SCK: track 0.00 -> 22.9 mm, vias 0 -> 1
- net Net-(J6-Pin_5): track 25.9 -> 47.1 mm
- net Net-(BZ1--): track 35.4 -> 15.1 mm
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Other:
- board text added: "L8 - levelator v0.0.2"
- board text removed: "L8 - XXXXXXXX062024"
