File: sensor.kicad_sch (KiCad schematic)
At the start: 20 parts, among them Q1 SI2301CDS-T1-GE3, U4 ST_SENSOR_2, U5 IIS3DHHCTR

Commit message: usb sheet
Parts:
- U4, U5: now not fitted
Changed lines of the file:
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@@
 		(in_bom yes)
 		(on_board yes)
-		(dnp no)
+		(dnp yes)
 		(fields_autoplaced yes)
 		(property "Reference" "U4"
@@
 		(in_bom yes)
 		(on_board yes)
-		(dnp no)
+		(dnp yes)
 		(fields_autoplaced yes)
 		(property "Reference" "U5"

Commit message: smaller test pads
Parts:
- removed D8: LED-YELLOW, LED_SMD:LED_0603_1608Metric, symbol Device:LED
- removed R30: 100R, Resistor_SMD:R_0603_1608Metric, symbol Device:R
- R13: value R100 -> 100R; LCSC (none) -> C22775
- TP3, TP4, TP5: footprint TestPoint:TestPoint_Pad_D1.0mm -> dnt:TestPoint_Pad_D1.0mm FP .6R

Commit message: pre-quilter after cap size issue
Parts:
- removed C3: 100nF, Capacitor_SMD:C_01005_0402Metric, symbol Device:C
- C2: footprint Capacitor_SMD:C_01005_0402Metric -> Capacitor_SMD:C_0603_1608Metric; LCSC C1525 -> (none); Manufacturer Samsung -> (none); Voltage 16V -> (none)
Other:
- moved on the sheet: C10
Changed lines of the file:
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@@
 	)
 	(junction
-		(at 132.08 109.22)
-		(diameter 0)
-		(color 0 0 0 0)
-	)
-	(junction
 		(at 139.7 109.22)
 		(diameter 0)
@@
 	)
 	(junction
-		(at 181.61 24.13)
-		(diameter 0)
-		(color 0 0 0 0)
-	)
-	(junction
-		(at 132.08 52.07)
+		(at 173.99 24.13)
 		(diameter 0)
 		(color 0 0 0 0)
@@
 	)
 	(junction
-		(at 181.61 109.22)
+		(at 173.99 109.22)
 		(diameter 0)
 		(color 0 0 0 0)
@@
 	(wire
 		(pts
-			(xy 132.08 52.07) (xy 132.08 68.58)
-		)
-		(stroke
-			(width 0)
-			(type default)
-		)
-	)
-	(wire
-		(pts
 			(xy 198.12 55.88) (xy 201.93 55.88)
 		)
@@
 	(wire
 		(pts
-			(xy 124.46 109.22) (xy 132.08 109.22)
+			(xy 124.46 109.22) (xy 139.7 109.22)
 		)
 		(stroke
@@
 	(wire
 		(pts
-			(xy 181.61 109.22) (xy 241.3 109.22)
+			(xy 173.99 109.22) (xy 241.3 109.22)
 		)
 		(stroke
@@
 	(wire
 		(pts
-			(xy 198.12 24.13) (xy 181.61 24.13)
+			(xy 198.12 24.13) (xy 173.99 24.13)
 		)
 		(stroke
@@
 	(wire
 		(pts
-			(xy 168.91 109.22) (xy 181.61 109.22)
+			(xy 168.91 109.22) (xy 173.99 109.22)
 		)
 		(stroke
@@
 	(wire
 		(pts
-			(xy 181.61 24.13) (xy 181.61 39.37)
+			(xy 173.99 24.13) (xy 173.99 39.37)
 		)
 		(stroke
@@
 	(wire
 		(pts
-			(xy 168.91 24.13) (xy 181.61 24.13)
+			(xy 168.91 24.13) (xy 173.99 24.13)
 		)
 		(stroke
@@
 	(wire
 		(pts
-			(xy 132.08 76.2) (xy 132.08 109.22)
-		)
-		(stroke
-			(width 0)
-			(type default)
-		)
-	)
-	(wire
-		(pts
 			(xy 139.7 57.15) (xy 149.86 57.15)
 		)
@@
 	(wire
 		(pts
-			(xy 132.08 109.22) (xy 139.7 109.22)
-		)
-		(stroke
-			(width 0)
-			(type default)
-		)
-	)
-	(wire
-		(pts
 			(xy 124.46 77.47) (xy 124.46 80.01)
 		)
@@
 	(wire
 		(pts
-			(xy 181.61 46.99) (xy 181.61 109.22)
+			(xy 173.99 46.99) (xy 173.99 109.22)
 		)
 		(stroke
@@
 	)
 	(symbol
-		(lib_id "Device:C")
-		(at 132.08 72.39 0)
-		(unit 1)
-		(exclude_from_sim no)
-		(in_bom yes)
-		(on_board yes)
-		(dnp no)
-		(property "Reference" "C3"
-			(at 133.35 71.12 90)
-			(effects
-				(font
-					(size 1.27 1.27)
-				)
-				(justify left)
-			)
-		)
-		(property "Value" "100nF"
-			(at 133.35 80.01 90)
-			(effects
-				(font
-					(size 1.27 1.27)
-				)
-				(justify left)
-			)
-		)
-		(property "Footprint" "Capacitor_SMD:C_01005_0402Metric"
-			(at 12.192 31.75 90)
-			(effects
-				(font
-					(size 1.524 1.524)
-				)
-				(hide yes)
-			)
-		)
-		(property "Datasheet" "~"
-			(at 132.08 72.39 0)
-			(effects
-				(font
-					(size 1.524 1.524)
-				)
-				(hide yes)
-			)
-		)
-		(property "Description" "Unpolarized capacitor X7R"
-			(at 132.08 72.39 0)
-			(effects
-				(font
-					(size 1.27 1.27)
-				)
-				(hide yes)
-			)
-		)
-		(property "LCSC" "C1525"
-			(at 132.08 72.39 0)
-			(effects
-				(font
-					(size 1.27 1.27)
-				)
-				(hide yes)
-			)
-		)
-		(property "Manufacturer" "Samsung"
-			(at 132.08 72.39 0)
-			(effects
-				(font
-					(size 1.27 1.27)
-				)
-				(hide yes)
-			)
-		)
-		(property "Sim.Device" ""
-			(at 132.08 72.39 0)
-			(effects
-				(font
-					(size 1.27 1.27)
-				)
-				(hide yes)
-			)
-		)
-		(property "Sim.Pins" ""
-			(at 132.08 72.39 0)
-			(effects
-				(font
-					(size 1.27 1.27)
-				)
-				(hide yes)
-			)
-		)
-		(property "Voltage" "16V"
-			(at 132.08 72.39 90)
-			(effects
-				(font
-					(size 1.27 1.27)
-				)
-				(hide yes)
-			)
-		)
-		(property "Silkscreen" ""
-			(at 132.08 72.39 0)
-			(effects
-				(font
-					(size 1.27 1.27)
-				)
-				(hide yes)
-			)
-		)
-		(pin "1"
-		)
-		(pin "2"
-		)
-		(instances
-			(project "l8-kicad"
-				(path "/8d063f79-9282-4820-bcf4-1ff3c006cf08/801ffdec-7184-42a0-bbdb-64e97598ca97"
-					(reference "C3")
-					(unit 1)
-				)
-			)
-		)
-	)
-	(symbol
 		(lib_id "dnt:ST_SENSOR_2")
 		(at 226.06 43.18 0)
@@
 	(symbol
 		(lib_id "Device:C")
-		(at 181.61 43.18 0)
+		(at 173.99 43.18 0)
 		(unit 1)
 		(exclude_from_sim no)
@@
 		(dnp no)
 		(property "Reference" "C10"
-			(at 184.531 42.0116 0)
+			(at 176.911 42.0116 0)
 			(effects
 				(font
@@
 		)
 		(property "Value" "10uF"
-			(at 184.15 44.45 0)
+			(at 176.53 44.45 0)
 			(effects
 				(font
@@
 		)
 		(property "Footprint" "Capacitor_SMD:C_0805_2012Metric"
-			(at 182.5752 46.99 0)
+			(at 174.9552 46.99 0)
 			(effects
 				(font
@@
 		)
 		(property "Datasheet" ""
-			(at 181.61 43.18 0)
+			(at 173.99 43.18 0)
 			(effects
 				(font
@@
 		)
 		(property "Description" "X5R"
-			(at 181.61 43.18 0)
+			(at 173.99 43.18 0)
 			(effects
 				(font
@@
 		)
 		(property "PN" ""
-			(at 181.61 43.18 0)
+			(at 173.99 43.18 0)
 			(effects
 				(font
@@
 		)
 		(property "LCSC" "C96446"
-			(at 181.61 43.18 0)
+			(at 173.99 43.18 0)
 			(effects
 				(font
@@
 		)
 		(property "Voltage" "25V"
-			(at 186.69 46.99 0)
+			(at 179.07 46.99 0)
 			(effects
 				(font
@@
 		)
 		(property "Sim.Device" ""
-			(at 181.61 43.18 0)
+			(at 173.99 43.18 0)
 			(effects
 				(font
@@
 		)
 		(property "Sim.Pins" ""
-			(at 181.61 43.18 0)
+			(at 173.99 43.18 0)
 			(effects
 				(font
@@
 		)
 		(property "Silkscreen" ""
-			(at 181.61 43.18 0)
+			(at 173.99 43.18 0)
 			(effects
 				(font
@@
 			)
 		)
-		(property "Footprint" "Capacitor_SMD:C_01005_0402Metric"
+		(property "Footprint" "Capacitor_SMD:C_0603_1608Metric"
 			(at 49.022 8.89 90)
 			(effects
@@
 			)
 		)
-		(property "LCSC" "C1525"
+		(property "LCSC" ""
 			(at 168.91 49.53 0)
 			(effects
@@
 			)
 		)
-		(property "Manufacturer" "Samsung"
+		(property "Manufacturer" ""
 			(at 168.91 49.53 0)
 			(effects
@@
 			)
 		)
-		(property "Voltage" "16V"
+		(property "Voltage" ""
 			(at 168.91 49.53 90)
 			(effects

Commit message: pre JLCPCB try 1
Parts:
- C2: LCSC (none) -> C14663
- TP3, TP5, U4, U5: now left out of the parts list
- TP4: Manufacturer DNP -> (none); Part # DNP -> (none); VEND DNP -> (none); VEND# DNP -> (none); now left out of the parts list
Changed lines of the file:
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@@
 		(unit 1)
 		(exclude_from_sim no)
-		(in_bom yes)
+		(in_bom no)
 		(on_board yes)
 		(dnp yes)
@@
 		(unit 1)
 		(exclude_from_sim no)
-		(in_bom yes)
+		(in_bom no)
 		(on_board yes)
 		(dnp no)
@@
 			)
 		)
-		(property "LCSC" ""
+		(property "LCSC" "C14663"
 			(at 168.91 49.53 0)
 			(effects
@@
 		(unit 1)
 		(exclude_from_sim no)
-		(in_bom yes)
+		(in_bom no)
 		(on_board yes)
 		(dnp yes)
@@
 		(unit 1)
 		(exclude_from_sim no)
-		(in_bom yes)
+		(in_bom no)
 		(on_board yes)
 		(dnp no)
@@
 		(unit 1)
 		(exclude_from_sim no)
-		(in_bom yes)
+		(in_bom no)
 		(on_board yes)
 		(dnp no)
@@
 			)
 		)
-		(property "Part #" "DNP"
+		(property "Part #" ""
 			(at 208.915 295.91 0)
 			(effects
@@
 			)
 		)
-		(property "VEND" "DNP"
+		(property "VEND" ""
 			(at 208.915 295.91 0)
 			(effects
@@
 			)
 		)
-		(property "VEND#" "DNP"
+		(property "VEND#" ""
 			(at 208.915 295.91 0)
 			(effects
@@
 			)
 		)
-		(property "Manufacturer" "DNP"
+		(property "Manufacturer" ""
 			(at 208.915 295.91 0)
 			(effects

Commit message: version 2 changes
Parts:
- U4: footprint Package_DIP:DIP-24_W15.24mm_Socket -> dnt:DIP-24_W15.24mm_Socket- nox
Changed lines of the file:
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@@
 	)
 	(symbol
-		(lib_id "l8-kicad-rescue:PWR_FLAG-power")
+		(lib_id "power:PWR_FLAG")
 		(at 278.13 109.22 0)
 		(unit 1)
@@
 			)
 		)
-		(property "Datasheet" ""
+		(property "Datasheet" "~"
 			(at 278.13 109.22 0)
 			(effects
@@
 			)
 		)
-		(property "Description" ""
+		(property "Description" "Special symbol for telling ERC where power comes from"
 			(at 278.13 109.22 0)
 			(effects
@@
 			)
 		)
-		(property "Footprint" "Package_DIP:DIP-24_W15.24mm_Socket"
+		(property "Footprint" "dnt:DIP-24_W15.24mm_Socket- nox"
 			(at 226.06 43.18 0)
 			(effects
@@
 	)
 	(symbol
-		(lib_id "l8-kicad-rescue:GND-power")
+		(lib_id "power:GND")
 		(at 73.66 132.08 0)
 		(unit 1)
@@
 	)
 	(symbol
-		(lib_id "l8-kicad-rescue:GND-power")
+		(lib_id "power:GND")
 		(at 96.52 130.81 0)
 		(unit 1)

Commit message: x
Parts:
- removed Q1: SI2301CDS-T1-GE3, Package_TO_SOT_SMD:SOT-23, symbol dnt:SI2301CDS-T1-GE3
- added Q1: AO3400A, Package_TO_SOT_SMD:SOT-23, symbol dnt:AO3400A
Connections:
- net GND: now also Q1.2 (S)
- net at C10.2, C2.2, R10.1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: now also Q1.3 (D)
- net at R13.2, R2.2: now also Q1.1 (G)
Changed lines of the file:
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@@
+	)
+	(symbol
+		(lib_id "dnt:AO3400A")
+		(at 93.98 116.84 0)
+		(unit 1)
+		(exclude_from_sim no)
+		(in_bom yes)
+		(on_board yes)
+		(dnp no)
+		(fields_autoplaced yes)
+		(property "Reference" "Q1"
+			(at 100.33 115.5699 0)
+			(effects
+				(font
+					(size 1.27 1.27)
+				)
+				(justify left)
+			)
+		)
+		(property "Value" "AO3400A"
+			(at 100.33 118.1099 0)
+			(effects
+				(font
+					(size 1.27 1.27)
+				)
+				(justify left)
+			)
+		)
+		(property "Footprint" "Package_TO_SOT_SMD:SOT-23"
+			(at 99.06 118.745 0)
+			(effects
+				(font
+					(size 1.27 1.27)
+					(italic yes)
+				)
+				(justify left)
+				(hide yes)
+			)
+		)
+		(property "Datasheet" "http://www.aosmd.com/pdfs/datasheet/AO3400A.pdf"
+			(at 99.06 120.65 0)
+			(effects
+				(font
+					(size 1.27 1.27)
+				)
+				(justify left)
+				(hide yes)
+			)
+		)
+		(property "Description" "30V Vds, 5.7A Id, N-Channel MOSFET, SOT-23"
+			(at 93.98 116.84 0)
+			(effects
+				(font
+					(size 1.27 1.27)
+				)
+				(hide yes)
+			)
+		)
+		(pin "2"
+		)
+		(pin "1"
+		)
+		(pin "3"
+		)
+		(instances
+			(project ""
+				(path "/8d063f79-9282-4820-bcf4-1ff3c006cf08/801ffdec-7184-42a0-bbdb-64e97598ca97"
+					(reference "Q1")
+					(unit 1)
+				)
+			)
+		)
 	)
 	(symbol
@@
 					(unit 1)
 				)
-			)
-		)
-	)
-	(symbol
-		(lib_id "dnt:SI2301CDS-T1-GE3")
-		(at 93.98 116.84 0)
-		(unit 1)
-		(exclude_from_sim no)
-		(in_bom yes)
-		(on_board yes)
-		(dnp no)
-		(fields_autoplaced yes)
-		(property "Reference" "Q1"
-			(at 100.33 115.5699 0)
-			(effects
-				(font
-					(size 1.27 1.27)
-				)
-				(justify left)
-			)
-		)
-		(property "Value" "SI2301CDS-T1-GE3"
-			(at 100.33 118.1099 0)
-			(effects
-				(font
-					(size 1.27 1.27)
-				)
-				(justify left)
-			)
-		)
-		(property "Footprint" "Package_TO_SOT_SMD:SOT-23"
-			(at 100.33 118.745 0)
-			(effects
-				(font
-					(size 1.27 1.27)
-					(italic yes)
-				)
-				(justify left)
-				(hide yes)
-			)
-		)
-		(property "Datasheet" "https://wmsc.lcsc.com/wmsc/upload/file/pdf/v2/lcsc/1808272021_Vishay-Intertech-SI2301CDS-T1-GE3_C10487.pdf"
-			(at 93.98 116.84 0)
-			(effects
-				(font
-					(size 1.27 1.27)
-				)
-				(justify left)
-				(hide yes)
-			)
-		)
-		(property "Description" "Generic N-Channel Power MOSFET"
-			(at 93.98 116.84 0)
-			(effects
-				(font
-					(size 1.27 1.27)
-				)
-				(hide yes)
-			)
-		)
-		(property "LCSC" " C20917"
-			(at 102.87 116.84 0)
-			(effects
-				(font
-					(size 1.27 1.27)
-				)
-				(hide yes)
-			)
-		)
-		(property "Sim.Device" ""
-			(at 93.98 116.84 0)
-			(effects
-				(font
-					(size 1.27 1.27)
-				)
-				(hide yes)
-			)
-		)
-		(property "Sim.Pins" ""
-			(at 93.98 116.84 0)
-			(effects
-				(font
-					(size 1.27 1.27)
-				)
-				(hide yes)
-			)
-		)
-		(property "Silkscreen" ""
-			(at 93.98 116.84 0)
-			(effects
-				(font
-					(size 1.27 1.27)
-				)
-				(hide yes)
-			)
-		)
-		(pin "2"
-		)
-		(pin "1"
-		)
-		(pin "3"
-		)
-		(instances
-			(project "l8-kicad"
-				(path "/8d063f79-9282-4820-bcf4-1ff3c006cf08/801ffdec-7184-42a0-bbdb-64e97598ca97"
-					(reference "Q1")
-					(unit 1)
-				)

Commit message: version 2 initial
Connections:
- net GND: now also C10.2, C2.2, R10.1, R11.1, R12.1, R9.1
- net at Q1.3 (D), U4.13 (GND), U5.10 (GND__1)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: no longer C10.2, C2.2, R10.1, R11.1, R12.1, R9.1
Other:
- moved on the sheet: C10, C2, R10, R8, R9

Commit message: SENT TO jlcpcb
Parts:
- C10: footprint Capacitor_SMD:C_0805_2012Metric -> Capacitor_SMD:C_0603_1608Metric
Connections:
- net +3.3V renamed +3.3VP
Other:
- note added: "LIS3DHHTR C2655077 CCLGA-16(5x5)"
Changed lines of the file:
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@@
+		)
+	)
+	(text "LIS3DHHTR\n  C2655077 \n  CCLGA-16(5x5)\n\n"
+		(exclude_from_sim no)
+		(at 102.362 202.946 0)
+		(effects
+			(font
+				(size 10.16 10.16)
+			)
 		)
 	)
@@
 			)
 			(justify left)
-		)
-	)
-	(netclass_flag ""
-		(length 2.54)
-		(shape round)
-		(at 71.12 24.13 0)
-		(effects
-			(font
-				(size 1.27 1.27)
-			)
-			(justify left bottom)
-		)
-		(property "Netclass" "3.3V"
-			(at 72.136 19.304 0)
-			(show_name yes)
-			(effects
-				(font
-					(size 1.27 1.27)
-					(italic yes)
-				)
-				(justify left)
-			)
 		)
 	)
@@
 	)
 	(symbol
+		(lib_id "power:+3.3VP")
+		(at 38.1 24.13 0)
+		(unit 1)
+		(exclude_from_sim no)
+		(in_bom yes)
+		(on_board yes)
+		(dnp no)
+		(fields_autoplaced yes)
+		(property "Reference" "#PWR09"
+			(at 41.91 25.4 0)
+			(effects
+				(font
+					(size 1.27 1.27)
+				)
+				(hide yes)
+			)
+		)
+		(property "Value" "+3.3VP"
+			(at 38.1 19.05 0)
+			(effects
+				(font
+					(size 1.27 1.27)
+				)
+			)
+		)
+		(property "Footprint" ""
+			(at 38.1 24.13 0)
+			(effects
+				(font
+					(size 1.27 1.27)
+				)
+				(hide yes)
+			)
+		)
+		(property "Datasheet" ""
+			(at 38.1 24.13 0)
+			(effects
+				(font
+					(size 1.27 1.27)
+				)
+				(hide yes)
+			)
+		)
+		(property "Description" "Power symbol creates a global label with name \"+3.3VP\""
+			(at 38.1 24.13 0)
+			(effects
+				(font
+					(size 1.27 1.27)
+				)
+				(hide yes)
+			)
+		)
+		(pin "1"
+		)
+		(instances
+			(project ""
+				(path "/8d063f79-9282-4820-bcf4-1ff3c006cf08/801ffdec-7184-42a0-bbdb-64e97598ca97"
+					(reference "#PWR09")
+					(unit 1)
+				)
+			)
+		)
+	)
+	(symbol
 		(lib_id "power:GND")
 		(at 173.99 143.51 0)
@@
 			)
 		)
-		(property "Footprint" "Capacitor_SMD:C_0805_2012Metric"
+		(property "Footprint" "Capacitor_SMD:C_0603_1608Metric"
 			(at 116.5352 41.91 0)
 			(effects
@@
 	)
 	(symbol
-		(lib_id "power:+3.3V")
-		(at 38.1 24.13 0)
-		(unit 1)
-		(exclude_from_sim no)
-		(in_bom yes)
-		(on_board yes)
-		(dnp no)
-		(fields_autoplaced yes)
-		(property "Reference" "#PWR09"
-			(at 38.1 27.94 0)
-			(effects
-				(font
-					(size 1.27 1.27)
-				)
-				(hide yes)
-			)
-		)
-		(property "Value" "+3.3V"
-			(at 38.1 19.05 0)
-			(effects
-				(font
-					(size 1.27 1.27)
-				)
-			)
-		)
-		(property "Footprint" ""
-			(at 38.1 24.13 0)
-			(effects
-				(font
-					(size 1.27 1.27)
-				)
-				(hide yes)
-			)
-		)
-		(property "Datasheet" ""
-			(at 38.1 24.13 0)
-			(effects
-				(font
-					(size 1.27 1.27)
-				)
-				(hide yes)
-			)
-		)
-		(property "Description" "Power symbol creates a global label with name \"+3.3V\""
-			(at 38.1 24.13 0)
-			(effects
-				(font
-					(size 1.27 1.27)
-				)
-				(hide yes)
-			)
-		)
-		(pin "1"
-		)
-		(instances
-			(project "l8-kicad"
-				(path "/8d063f79-9282-4820-bcf4-1ff3c006cf08/801ffdec-7184-42a0-bbdb-64e97598ca97"
-					(reference "#PWR09")
-					(unit 1)
-				)
-			)
-		)
-	)
-	(symbol
 		(lib_id "Device:R")
 		(at 260.35 59.69 0)
@@
 			)
 		)
-		(property "Description" "Unpolarized capacitor X7R"
+		(property "Description" "50V 100nF X7R ±10% 0603 Multilayer Ceramic Capacitors MLCC - SMD/SMT ROHS"
 			(at 110.49 38.1 0)
 			(effects
