File: usb.kicad_sch (KiCad schematic)
At the start: 9 parts, among them J1 USB_B_Mini

Commit message: smaller test pads
Parts:
- removed D7: LED-YELLOW, LED_SMD:LED_0603_1608Metric, symbol Device:LED
- removed R6: 1K, Resistor_SMD:R_0603_1608Metric, symbol Device:R
Other:
- note removed: "USB power"

Commit message: pre-quilter after cap size issue
Parts:
- C6: footprint Capacitor_SMD:C_01005_0402Metric -> Capacitor_SMD:C_0603_1608Metric; LCSC C1525 -> (none); Manufacturer Samsung -> (none); Voltage 16V -> (none)
- D10: footprint Package_TO_SOT_SMD:SOT-363_SC-70-6 -> Package_TO_SOT_SMD:SOT-23-6; LCSC C85364 -> C2836319
Changed lines of the file:
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@@
 			)
 		)
-		(property "Footprint" "Capacitor_SMD:C_01005_0402Metric"
+		(property "Footprint" "Capacitor_SMD:C_0603_1608Metric"
 			(at -8.128 67.31 90)
 			(effects
@@
 			)
 		)
-		(property "LCSC" "C1525"
-			(at 111.76 107.95 0)
-			(effects
-				(font
-					(size 1.27 1.27)
-				)
-				(hide yes)
-			)
-		)
-		(property "Manufacturer" "Samsung"
+		(property "LCSC" ""
+			(at 111.76 107.95 0)
+			(effects
+				(font
+					(size 1.27 1.27)
+				)
+				(hide yes)
+			)
+		)
+		(property "Manufacturer" ""
 			(at 111.76 107.95 0)
 			(effects
@@
 			)
 		)
-		(property "Voltage" "16V"
+		(property "Voltage" ""
 			(at 111.76 107.95 90)
 			(effects
@@
 			)
 		)
-		(property "Footprint" "Package_TO_SOT_SMD:SOT-363_SC-70-6"
+		(property "Footprint" "Package_TO_SOT_SMD:SOT-23-6"
 			(at 151.13 110.49 0)
 			(effects
@@
 			)
 		)
-		(property "Datasheet" "http://www.onsemi.com/pub_link/Collateral/NUP4202W1-D.PDF"
+		(property "Datasheet" ""
 			(at 151.13 101.6 90)
 			(effects
@@
 			)
 		)
-		(property "Description" "Transient voltage suppressor designed to protect high speed data lines from ESD, EFT, and lightning"
+		(property "Description" ""
 			(at 151.13 101.6 0)
 			(effects
@@
 			)
 		)
-		(property "LCSC" "C85364"
+		(property "LCSC" "C2836319"
 			(at 151.13 101.6 0)
 			(effects

Commit message: pre JLCPCB try 1
Parts:
- C6: LCSC (none) -> C14663
Changed lines of the file:
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@@
 			)
 		)
-		(property "LCSC" ""
+		(property "LCSC" "C14663"
 			(at 111.76 107.95 0)
 			(effects

Commit message: SENT TO jlcpcb
Parts:
- D10: JLCPCB Rotation Offset (none) -> 90
- D12: JLCPCB Rotation Offset (none) -> 180
Changed lines of the file:
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@@
+			)
+		)
+		(property "JLCPCB Rotation Offset" "180"
+			(at 156.21 78.74 0)
+			(effects
+				(font
+					(size 1.27 1.27)
+				)
+				(hide yes)
 			)
 		)
@@
 			(at 151.13 101.6 0)
 			(effects
+				(font
+					(size 1.27 1.27)
+				)
+				(hide yes)
+			)
+		)
+		(property "JLCPCB Rotation Offset" "90"
+			(at 151.13 101.6 0)
+			(effects

Commit message: x
Parts:
- D12: footprint Diode_SMD:D_SOD-123 -> dnt:D_SOD-123-polarity
Changed lines of the file:
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@@
 			)
 		)
-		(property "Footprint" "Diode_SMD:D_SOD-123"
+		(property "Footprint" "dnt:D_SOD-123-polarity"
 			(at 97.79 -219.583 90)
 			(effects

Commit message: version 2 initial
Other:
- moved on the sheet: C6, R5

Commit message: SENT TO jlcpcb
Parts:
- D12: JLCPCB Rotation Offset 180 -> 0
- J1: now not fitted
Changed lines of the file:
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@@
 			)
 		)
-		(property "Description" "Unpolarized capacitor X7R"
+		(property "Description" "50V 100nF X7R ±10% 0603 Multilayer Ceramic Capacitors MLCC - SMD/SMT ROHS"
 			(at 86.36 106.68 0)
 			(effects
@@
 			)
 		)
-		(property "JLCPCB Rotation Offset" "180"
+		(property "JLCPCB Rotation Offset" "0"
 			(at 156.21 78.74 0)
 			(effects
@@
 		(in_bom yes)
 		(on_board yes)
-		(dnp no)
+		(dnp yes)
 		(fields_autoplaced yes)
 		(property "Reference" "J1"
