File: usb.kicad_sch (KiCad schematic)
At the start: 7 parts, among them J1 USB_B_Mini

Commit message: update to version 9 on selwyn
Other:
- title: (none) -> l8
Changed lines of the file:
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@@
 (kicad_sch
-	(version 20231120)
+	(version 20250114)
 	(generator "eeschema")
-	(generator_version "8.0")
+	(generator_version "9.0")
 	(paper "A4")
+	(title_block
+		(title "l8")
+	)
 	(junction
 		(at 153.67 82.55)
@@
 	(label "Shield"
 		(at 81.28 100.33 180)
-		(fields_autoplaced yes)
 		(effects
 			(font
@@
 		(shape output)
 		(at 245.11 82.55 0)
-		(fields_autoplaced yes)
 		(effects
 			(font
@@
 		(shape bidirectional)
 		(at 175.26 90.17 0)
-		(fields_autoplaced yes)
 		(effects
 			(font
@@
 		(shape bidirectional)
 		(at 175.26 92.71 0)
-		(fields_autoplaced yes)
 		(effects
 			(font
@@
 		(shape bidirectional)
 		(at 175.26 87.63 0)
-		(fields_autoplaced yes)
-		(effects
-			(font
+		(effects
+			(font
