File: lcd.kicad_sch (KiCad schematic)
At the start: 7 parts, among them J2 LCD 3.2" 240x320 Conn_01x14_P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, Q4 SI2301CDS-T1-GE3

Commit message: version 2 changes
Other:
- moved on the sheet: R39
Changed lines of the file:
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@@
 	)
 	(junction
-		(at 195.58 71.12)
+		(at 194.31 71.12)
 		(diameter 0)
 		(color 0 0 0 0)
@@
 	(wire
 		(pts
-			(xy 135.89 60.96) (xy 140.97 60.96)
+			(xy 135.89 60.96) (xy 238.76 60.96)
 		)
 		(stroke
@@
 	(wire
 		(pts
-			(xy 135.89 71.12) (xy 195.58 71.12)
-		)
-		(stroke
-			(width 0)
-			(type default)
-		)
-	)
-	(wire
-		(pts
-			(xy 135.89 58.42) (xy 140.97 58.42)
+			(xy 135.89 71.12) (xy 194.31 71.12)
+		)
+		(stroke
+			(width 0)
+			(type default)
+		)
+	)
+	(wire
+		(pts
+			(xy 135.89 58.42) (xy 238.76 58.42)
 		)
 		(stroke
@@
 	(wire
 		(pts
-			(xy 180.34 50.8) (xy 201.93 50.8)
+			(xy 180.34 50.8) (xy 238.76 50.8)
 		)
 		(stroke
@@
 	(wire
 		(pts
-			(xy 195.58 67.31) (xy 195.58 71.12)
-		)
-		(stroke
-			(width 0)
-			(type default)
-		)
-	)
-	(wire
-		(pts
-			(xy 135.89 66.04) (xy 140.97 66.04)
-		)
-		(stroke
-			(width 0)
-			(type default)
-		)
-	)
-	(wire
-		(pts
-			(xy 135.89 78.74) (xy 140.97 78.74)
-		)
-		(stroke
-			(width 0)
-			(type default)
-		)
-	)
-	(wire
-		(pts
-			(xy 135.89 55.88) (xy 140.97 55.88)
+			(xy 194.31 49.53) (xy 194.31 71.12)
+		)
+		(stroke
+			(width 0)
+			(type default)
+		)
+	)
+	(wire
+		(pts
+			(xy 135.89 66.04) (xy 238.76 66.04)
+		)
+		(stroke
+			(width 0)
+			(type default)
+		)
+	)
+	(wire
+		(pts
+			(xy 135.89 78.74) (xy 238.76 78.74)
+		)
+		(stroke
+			(width 0)
+			(type default)
+		)
+	)
+	(wire
+		(pts
+			(xy 135.89 55.88) (xy 238.76 55.88)
 		)
 		(stroke
@@
 	(wire
 		(pts
-			(xy 135.89 73.66) (xy 140.97 73.66)
-		)
-		(stroke
-			(width 0)
-			(type default)
-		)
-	)
-	(wire
-		(pts
-			(xy 135.89 76.2) (xy 140.97 76.2)
+			(xy 135.89 73.66) (xy 238.76 73.66)
+		)
+		(stroke
+			(width 0)
+			(type default)
+		)
+	)
+	(wire
+		(pts
+			(xy 135.89 76.2) (xy 238.76 76.2)
 		)
 		(stroke
@@
 	(wire
 		(pts
-			(xy 135.89 63.5) (xy 140.97 63.5)
+			(xy 194.31 71.12) (xy 238.76 71.12)
+		)
+		(stroke
+			(width 0)
+			(type default)
+		)
+	)
+	(wire
+		(pts
+			(xy 135.89 63.5) (xy 238.76 63.5)
 		)
 		(stroke
@@
 	(wire
 		(pts
-			(xy 195.58 59.69) (xy 195.58 27.94)
-		)
-		(stroke
-			(width 0)
-			(type default)
-		)
-	)
-	(wire
-		(pts
-			(xy 195.58 27.94) (xy 187.96 27.94)
-		)
-		(stroke
-			(width 0)
-			(type default)
-		)
-	)
-	(wire
-		(pts
-			(xy 187.96 53.34) (xy 201.93 53.34)
-		)
-		(stroke
-			(width 0)
-			(type default)
-		)
-	)
-	(wire
-		(pts
-			(xy 195.58 71.12) (xy 201.93 71.12)
+			(xy 194.31 41.91) (xy 194.31 27.94)
+		)
+		(stroke
+			(width 0)
+			(type default)
+		)
+	)
+	(wire
+		(pts
+			(xy 194.31 27.94) (xy 187.96 27.94)
+		)
+		(stroke
+			(width 0)
+			(type default)
+		)
+	)
+	(wire
+		(pts
+			(xy 187.96 53.34) (xy 238.76 53.34)
 		)
 		(stroke
@@
 	(wire
 		(pts
-			(xy 135.89 68.58) (xy 140.97 68.58)
+			(xy 135.89 68.58) (xy 238.76 68.58)
 		)
 		(stroke
@@
 	(hierarchical_label "LCD_SDI"
 		(shape input)
-		(at 140.97 58.42 0)
+		(at 238.76 58.42 0)
 		(fields_autoplaced yes)
 		(effects
@@
 	(hierarchical_label "LCD_LED"
 		(shape input)
-		(at 140.97 63.5 0)
+		(at 238.76 63.5 0)
 		(fields_autoplaced yes)
 		(effects
@@
 	(hierarchical_label "T_CS"
 		(shape input)
-		(at 201.93 71.12 0)
+		(at 238.76 71.12 0)
 		(fields_autoplaced yes)
 		(effects
@@
 	(hierarchical_label "T_IRQ"
 		(shape input)
-		(at 140.97 78.74 0)
+		(at 238.76 78.74 0)
 		(fields_autoplaced yes)
 		(effects
@@
 	(hierarchical_label "T_SDI"
 		(shape input)
-		(at 140.97 73.66 0)
+		(at 238.76 73.66 0)
 		(fields_autoplaced yes)
 		(effects
@@
 	(hierarchical_label "T_SDO"
 		(shape output)
-		(at 140.97 76.2 0)
+		(at 238.76 76.2 0)
 		(fields_autoplaced yes)
 		(effects
@@
 	(hierarchical_label "LCD_DC"
 		(shape input)
-		(at 140.97 55.88 0)
+		(at 238.76 55.88 0)
 		(fields_autoplaced yes)
 		(effects
@@
 	(hierarchical_label "T_CLK"
 		(shape input)
-		(at 140.97 68.58 0)
+		(at 238.76 68.58 0)
 		(fields_autoplaced yes)
 		(effects
@@
 	)
 	(hierarchical_label "LCD_SDO"
-		(shape output)
-		(at 140.97 66.04 0)
+		(shape tri_state)
+		(at 238.76 66.04 0)
 		(fields_autoplaced yes)
 		(effects
@@
 	(hierarchical_label "LCD_SCK"
 		(shape input)
-		(at 140.97 60.96 0)
+		(at 238.76 60.96 0)
 		(fields_autoplaced yes)
 		(effects
@@
 	(hierarchical_label "LCD_RESET"
 		(shape input)
-		(at 201.93 53.34 0)
+		(at 238.76 53.34 0)
 		(fields_autoplaced yes)
 		(effects
@@
 	(hierarchical_label "LCD_CS"
 		(shape input)
-		(at 201.93 50.8 0)
+		(at 238.76 50.8 0)
 		(fields_autoplaced yes)
 		(effects
@@
 	)
 	(symbol
-		(lib_id "l8-kicad-rescue:GND-power")
+		(lib_id "power:GND")
 		(at 157.48 118.11 0)
 		(unit 1)
@@
 	(symbol
 		(lib_id "Device:R")
-		(at 195.58 63.5 0)
+		(at 194.31 45.72 0)
 		(mirror x)
 		(unit 1)
@@
 		(dnp no)
 		(property "Reference" "R39"
-			(at 197.612 63.5 90)
+			(at 196.342 45.72 90)
 			(effects
 				(font
@@
 		)
 		(property "Value" "10K"
-			(at 195.58 63.5 90)
+			(at 194.31 45.212 90)
 			(effects
 				(font
@@
 		)
 		(property "Footprint" "Resistor_SMD:R_0603_1608Metric"
-			(at 254.762 121.92 90)
+			(at 253.492 104.14 90)
 			(effects
 				(font
@@
 		)
 		(property "Datasheet" "~"
-			(at 344.17 122.555 0)
+			(at 342.9 104.775 0)
 			(effects
 				(font
@@
 		)
 		(property "Description" "Resistor"
-			(at 195.58 63.5 0)
+			(at 194.31 45.72 0)
 			(effects
 				(font
@@
 		)
 		(property "Part #" ""
-			(at 77.47 -43.18 0)
+			(at 76.2 -60.96 0)
 			(effects
 				(font
@@
 		)
 		(property "VEND" ""
-			(at 77.47 -43.18 0)
+			(at 76.2 -60.96 0)
 			(effects
 				(font
@@
 		)
 		(property "VEND#" ""
-			(at 77.47 -43.18 0)
+			(at 76.2 -60.96 0)
 			(effects
 				(font
@@
 		)
 		(property "Manufacturer" ""
-			(at 77.47 -43.18 0)
+			(at 76.2 -60.96 0)
 			(effects
 				(font
@@
 		)
 		(property "LCSC" "C25804"
-			(at 195.58 63.5 0)
+			(at 194.31 45.72 0)
 			(effects
 				(font
@@
 		)
 		(property "Sim.Device" ""
-			(at 195.58 63.5 0)
+			(at 194.31 45.72 0)
 			(effects
 				(font
@@
 		)
 		(property "Sim.Pins" ""
-			(at 195.58 63.5 0)
+			(at 194.31 45.72 0)
 			(effects
 				(font
@@
 		)
 		(property "Silkscreen" ""
-			(at 195.58 63.5 0)
+			(at 194.31 45.72 0)
 			(effects
 				(font
@@
 	)
 	(symbol
-		(lib_id "l8-kicad-rescue:GND-power")
+		(lib_id "power:GND")
 		(at 134.62 119.38 0)
 		(unit 1)
@@
 	)
 	(symbol
-		(lib_id "l8-kicad-rescue:PWR_FLAG-power")
+		(lib_id "power:PWR_FLAG")
 		(at 148.59 95.25 0)
 		(unit 1)
@@
 			)
 		)
-		(property "Datasheet" ""
+		(property "Datasheet" "~"
 			(at 148.59 95.25 0)
 			(effects
@@
 			)
 		)
-		(property "Description" ""
+		(property "Description" "Special symbol for telling ERC where power comes from"
 			(at 148.59 95.25 0)
 			(effects

Commit message: x
Parts:
- removed Q4: SI2301CDS-T1-GE3, Package_TO_SOT_SMD:SOT-23, symbol dnt:SI2301CDS-T1-GE3
- added Q2: AO3400A, Package_TO_SOT_SMD:SOT-23, symbol dnt:AO3400A
Connections:
- net GND: now also Q2.2 (S)
- net at R14.2, R3.1: now also Q2.1 (G)
- net at J2.2 (GND): now also Q2.3 (D)
Changed lines of the file:
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@@
 	)
 	(symbol
-		(lib_id "dnt:SI2301CDS-T1-GE3")
+		(lib_id "dnt:AO3400A")
 		(at 154.94 104.14 0)
 		(unit 1)
@@
 		(dnp no)
 		(fields_autoplaced yes)
-		(property "Reference" "Q4"
+		(property "Reference" "Q2"
 			(at 161.29 102.8699 0)
 			(effects
@@
 			)
 		)
-		(property "Value" "SI2301CDS-T1-GE3"
+		(property "Value" "AO3400A"
 			(at 161.29 105.4099 0)
 			(effects
@@
 		)
 		(property "Footprint" "Package_TO_SOT_SMD:SOT-23"
-			(at 161.29 106.045 0)
+			(at 160.02 106.045 0)
 			(effects
 				(font
@@
 			)
 		)
-		(property "Datasheet" "https://wmsc.lcsc.com/wmsc/upload/file/pdf/v2/lcsc/1808272021_Vishay-Intertech-SI2301CDS-T1-GE3_C10487.pdf"
-			(at 154.94 104.14 0)
+		(property "Datasheet" "http://www.aosmd.com/pdfs/datasheet/AO3400A.pdf"
+			(at 160.02 107.95 0)
 			(effects
 				(font
@@
 			)
 		)
-		(property "Description" "Generic N-Channel Power MOSFET"
+		(property "Description" "30V Vds, 5.7A Id, N-Channel MOSFET, SOT-23"
 			(at 154.94 104.14 0)
 			(effects
@@
 			)
 		)
-		(property "LCSC" " C20917"
-			(at 163.83 104.14 0)
-			(effects
-				(font
-					(size 1.27 1.27)
-				)
-				(hide yes)
-			)
-		)
-		(property "Sim.Device" ""
-			(at 154.94 104.14 0)
-			(effects
-				(font
-					(size 1.27 1.27)
-				)
-				(hide yes)
-			)
-		)
-		(property "Sim.Pins" ""
-			(at 154.94 104.14 0)
-			(effects
-				(font
-					(size 1.27 1.27)
-				)
-				(hide yes)
-			)
-		)
-		(property "Silkscreen" ""
-			(at 154.94 104.14 0)
-			(effects
-				(font
-					(size 1.27 1.27)
-				)
-				(hide yes)
-			)
+		(pin "3"
 		)
 		(pin "2"
@@
 		(pin "1"
 		)
-		(pin "3"
-		)
 		(instances
-			(project "l8-kicad"
+			(project ""
 				(path "/8d063f79-9282-4820-bcf4-1ff3c006cf08/98bf8f66-79b9-41fc-9cd7-550fbae3319a"
-					(reference "Q4")
+					(reference "Q2")
 					(unit 1)
 				)

Commit message: version 2 initial
Parts:
- added J10: Conn_01x04_Pin, Connector_PinSocket_2.54mm:PinSocket_1x04_P2.54mm_Vertical, symbol Connector:Conn_01x04_Pin
- added J8: Conn_01x14_Pin, symbol Connector:Conn_01x14_Pin
- added J9: Conn_01x18_Pin, symbol Connector:Conn_01x18_Pin
- added JP1: Jumper_2_Small_Bridged, symbol Jumper:Jumper_2_Small_Bridged
- added JP3: SolderJumper_2_Open, Jumper:SolderJumper-2_P1.3mm_Open_TrianglePad1.0x1.5mm, symbol Jumper:SolderJumper_2_Open
- added JP4: SolderJumper_2_Bridged, Jumper:SolderJumper-2_P1.3mm_Open_TrianglePad1.0x1.5mm, symbol Jumper:SolderJumper_2_Bridged
- added Q4: NPN, symbol Simulation_SPICE:NPN
- added R22: 1k, Resistor_THT:R_Axial_DIN0207_L6.3mm_D2.5mm_P10.16mm_Horizontal, symbol PCM_SL_Resistors:1k
- added U7: SN74LVC1G14DRL, Package_TO_SOT_SMD:SOT-553, symbol 74xGxx:SN74LVC1G14DRL
- added U8: XC6206PxxxMR, Package_TO_SOT_SMD:SOT-23-3, symbol Regulator_Linear:XC6206PxxxMR
Connections:
- net T_CLK is gone; now on net LCD_SCK: J2.10 (T_SCK)
- net T_SDI is gone; now on net LCD_SDI: J2.12 (T_SDI)
- net T_SDO is gone; now on net LCD_SDO: J2.13 (T_SDO)
- net +3.3V: now also U7.5 (VCC)
- net GND: now also J8.2 (Pin_2), J9.17 (Pin_17), JP4.1 (A), Q4.3 (E), U7.3 (GND), U8.1 (GND)
- net at J2.2 (GND): now also JP3.2 (B), JP4.2 (B); no longer Q2.3 (D)
- net T_IRQ: no longer names the net of J2.14 (T_IRQ)
- net T_IRQ: now also U7.2
- new net: J9.1 (Pin_1), J9.10 (Pin_10), J9.11 (Pin_11), J9.12 (Pin_12), J9.2 (Pin_2), J9.3 (Pin_3), J9.4 (Pin_4), J9.5 (Pin_5), J9.6 (Pin_6), J9.7 (Pin_7), J9.8 (Pin_8), J9.9 (Pin_9)
- new net: J9.18 (Pin_18), JP1.2 (B), U8.2 (VO)
- new net: Q4.2 (B), R22.2
- new net: JP3.1 (A), Q2.3 (D)
- new net CS: J8.3 (Pin_3), J9.16 (Pin_16)
- new net LED: J8.8 (Pin_8), R22.1
- new net RESET: J8.4 (Pin_4), J9.15 (Pin_15)
- new net R/C: J8.5 (Pin_5)
- new net SCK: J8.7 (Pin_7)
- new net SDI: J8.6 (Pin_6), J9.13 (Pin_13), Q4.1 (C)
- new net SDO: J8.9 (Pin_9)
- new net SD_CS: J10.1 (Pin_1)
- new net SD_SCK: J10.4 (Pin_4)
- new net SD_SDI: J10.3 (Pin_3)
- new net SD_SDO: J10.2 (Pin_2)
- new net VCC: J8.1 (Pin_1), JP1.1 (A), U8.3 (VI)
- new net _T_IRQ: U7.4
- no-connect marks 0 -> 9
Other:
- note added: "Permanent LCD power"
- note added: "Pulled ? by LCD board?"
- note added: "This must be bridged - not use on 5V after making this mod!"
- moved on the sheet: J2, Q2, R14, R3, R37, R38, R39

Commit message: version 2 initial- fixes
Parts:
- J9: footprint (none) -> Connector_FFC-FPC:TE_1-84953-8_1x18-1MP_P1.0mm_Horizontal; now not fitted; now left out of the parts list
- JP3, JP4: now not fitted
Changed lines of the file:
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@@
 	(wire
 		(pts
-			(xy 186.69 121.92) (xy 220.98 121.92)
+			(xy 185.42 121.92) (xy 220.98 121.92)
 		)
 		(stroke
@@
 		)
 	)
-	(label "SD_CS"
-		(at 185.42 121.92 0)
-		(fields_autoplaced yes)
-		(effects
-			(font
-				(size 1.27 1.27)
-			)
-			(justify left bottom)
-		)
-	)
 	(label "GND"
 		(at 177.8 45.72 0)
@@
 		)
 	)
-	(label "SD_SCK"
-		(at 185.42 129.54 0)
-		(fields_autoplaced yes)
-		(effects
-			(font
-				(size 1.27 1.27)
-			)
-			(justify left bottom)
-		)
-	)
-	(label "SD_MOSI"
-		(at 185.42 124.46 0)
-		(fields_autoplaced yes)
-		(effects
-			(font
-				(size 1.27 1.27)
-			)
-			(justify left bottom)
-		)
-	)
 	(label "RESET"
 		(at 177.8 50.8 0)
@@
 	(label "LED"
 		(at 177.8 60.96 0)
-		(fields_autoplaced yes)
-		(effects
-			(font
-				(size 1.27 1.27)
-			)
-			(justify left bottom)
-		)
-	)
-	(label "SD_MISO"
-		(at 185.42 127 0)
 		(fields_autoplaced yes)
 		(effects
@@
 		(at 281.94 66.04 180)
 		(unit 1)
-		(exclude_from_sim no)
-		(in_bom yes)
-		(on_board yes)
-		(dnp no)
+		(exclude_from_sim yes)
+		(in_bom no)
+		(on_board no)
+		(dnp yes)
 		(fields_autoplaced yes)
 		(property "Reference" "J9"
@@
 			)
 		)
-		(property "Footprint" ""
+		(property "Footprint" "Connector_FFC-FPC:TE_1-84953-8_1x18-1MP_P1.0mm_Horizontal"
 			(at 281.94 66.04 0)
 			(effects
@@
 		(in_bom no)
 		(on_board yes)
-		(dnp no)
+		(dnp yes)
 		(fields_autoplaced yes)
 		(property "Reference" "JP4"
@@
 		(in_bom no)
 		(on_board yes)
-		(dnp no)
+		(dnp yes)
 		(fields_autoplaced yes)
 		(property "Reference" "JP3"

Commit message: SENT TO jlcpcb
Parts:
- J10: JLCPCB Rotation Offset (none) -> 90; LCSC (none) -> C7500773
- J2: now left out of the parts list
- U7: value SN74LVC1G14DRL -> SN74LVC1G14DRLR; LCSC (none) -> C2877550; Package (none) -> SOT-553
Connections:
- net +3.3V renamed +3.3VP
Changed lines of the file:
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@@
-	)
-	(symbol
-		(lib_id "power:+3.3V")
-		(at 64.77 25.4 0)
-		(unit 1)
-		(exclude_from_sim no)
-		(in_bom yes)
-		(on_board yes)
-		(dnp no)
-		(fields_autoplaced yes)
-		(property "Reference" "#PWR034"
-			(at 64.77 29.21 0)
-			(effects
-				(font
-					(size 1.27 1.27)
-				)
-				(hide yes)
-			)
-		)
-		(property "Value" "+3.3V"
-			(at 64.77 20.32 0)
-			(effects
-				(font
-					(size 1.27 1.27)
-				)
-			)
-		)
-		(property "Footprint" ""
-			(at 64.77 25.4 0)
-			(effects
-				(font
-					(size 1.27 1.27)
-				)
-				(hide yes)
-			)
-		)
-		(property "Datasheet" ""
-			(at 64.77 25.4 0)
-			(effects
-				(font
-					(size 1.27 1.27)
-				)
-				(hide yes)
-			)
-		)
-		(property "Description" "Power symbol creates a global label with name \"+3.3V\""
-			(at 64.77 25.4 0)
-			(effects
-				(font
-					(size 1.27 1.27)
-				)
-				(hide yes)
-			)
-		)
-		(pin "1"
-		)
-		(instances
-			(project "l8-kicad"
-				(path "/8d063f79-9282-4820-bcf4-1ff3c006cf08/98bf8f66-79b9-41fc-9cd7-550fbae3319a"
-					(reference "#PWR034")
-					(unit 1)
-				)
-			)
-		)
 	)
 	(symbol
@@
 	)
 	(symbol
+		(lib_id "power:+3.3VP")
+		(at 64.77 25.4 0)
+		(unit 1)
+		(exclude_from_sim no)
+		(in_bom yes)
+		(on_board yes)
+		(dnp no)
+		(fields_autoplaced yes)
+		(property "Reference" "#PWR032"
+			(at 68.58 26.67 0)
+			(effects
+				(font
+					(size 1.27 1.27)
+				)
+				(hide yes)
+			)
+		)
+		(property "Value" "+3.3VP"
+			(at 64.77 20.32 0)
+			(effects
+				(font
+					(size 1.27 1.27)
+				)
+			)
+		)
+		(property "Footprint" ""
+			(at 64.77 25.4 0)
+			(effects
+				(font
+					(size 1.27 1.27)
+				)
+				(hide yes)
+			)
+		)
+		(property "Datasheet" ""
+			(at 64.77 25.4 0)
+			(effects
+				(font
+					(size 1.27 1.27)
+				)
+				(hide yes)
+			)
+		)
+		(property "Description" "Power symbol creates a global label with name \"+3.3VP\""
+			(at 64.77 25.4 0)
+			(effects
+				(font
+					(size 1.27 1.27)
+				)
+				(hide yes)
+			)
+		)
+		(pin "1"
+		)
+		(instances
+			(project ""
+				(path "/8d063f79-9282-4820-bcf4-1ff3c006cf08/98bf8f66-79b9-41fc-9cd7-550fbae3319a"
+					(reference "#PWR032")
+					(unit 1)
+				)
+			)
+		)
+	)
+	(symbol
 		(lib_id "Device:R")
 		(at 58.42 129.54 0)
@@
 		(unit 1)
 		(exclude_from_sim no)
-		(in_bom yes)
+		(in_bom no)
 		(on_board yes)
 		(dnp yes)
@@
 			)
 		)
-		(property "Value" "SN74LVC1G14DRL"
+		(property "Value" "SN74LVC1G14DRLR"
 			(at 125.73 94.0114 0)
 			(effects
@@
 		)
 		(property "Description" "Single Schmitt NOT Gate, Low-Voltage CMOS, SOT-553"
+			(at 110.49 97.79 0)
+			(effects
+				(font
+					(size 1.27 1.27)
+				)
+				(hide yes)
+			)
+		)
+		(property "LCSC" "C2877550"
+			(at 110.49 97.79 0)
+			(effects
+				(font
+					(size 1.27 1.27)
+				)
+				(hide yes)
+			)
+		)
+		(property "Package" " SOT-553"
 			(at 110.49 97.79 0)
 			(effects
@@
 			(at 180.34 124.46 0)
 			(effects
+				(font
+					(size 1.27 1.27)
+				)
+				(hide yes)
+			)
+		)
+		(property "LCSC" "C7500773"
+			(at 180.34 124.46 0)
+			(effects
+				(font
+					(size 1.27 1.27)
+				)
+				(hide yes)
+			)
+		)
+		(property "JLCPCB Rotation Offset" "90"
+			(at 180.34 124.46 0)
+			(effects

Commit message: update to version 9 on selwyn
Other:
- title: (none) -> l8
