File: power.kicad_sch (KiCad schematic)
At the start: 13 parts, among them U1 B0505S-1WR2, U22 TLV76733DRVx

Commit message: version 2 changes
Parts:
- removed PS1: D36V6F5, Connector_PinHeader_2.54mm:PinHeader_1x04_P2.54mm_Vertical, symbol dnt:D36V6F5
- removed TP6: 5V ISO, dnt:TestPoint_Pad_D1.0mm FP .6R, symbol Connector:TestPoint
- added C3: 10uF, Capacitor_SMD:C_0805_2012Metric, symbol Device:C
- added D7: SS14, dnt:D_SMA - polarity, symbol Diode:B340
- added D8: LED-RED, LED_SMD:LED_0603_1608Metric, symbol Device:LED
- added F1, F2, F3: Fuse, Fuse:Fuse_0805_2012Metric, symbol Device:Fuse
- added L1: 3.3uH, Inductor_SMD:L_Sunlord_SWPA4030S, symbol Device:L_Ferrite
- added R20: 2.2K, Resistor_SMD:R_0603_1608Metric, symbol Device:R
- added U6: LMR14006, Package_TO_SOT_SMD:SOT-23-6, symbol Regulator_Switching:LMR14206
- D2: footprint Diode_SMD:D_SMA -> dnt:D_SMA - polarity
Connections:
- net +3.3V: now also F3.2; no longer C4.1, C5.2, C7.1, U22.1 (OUT), U22.2 (SNS)
- net +5V: now also D8.2 (A), F2.2
- net GND: now also C3.2, D7.2 (A), R20.1, U6.2 (GND)
- net VBATT: now also F1.1; no longer D2.2 (A)
- net at D1.2 (A), D2.1 (K), D3.1 (A1): now also C3.1, U6.5 (VIN)
- new net: C4.1, C5.2, C7.1, F3.1, U22.1 (OUT), U22.2 (SNS)
- new net: D2.2 (A), F1.2
- new net: D7.1 (K), L1.1, U6.6 (SW)
- new net: F2.1, L1.2
- new net: D8.1 (K), R20.2
- no-connect marks 2 -> 1
Other:
- moved on the sheet: C4, C5, C7, D1, D2, D3, R4, TP1, TP2, U1, U22

Commit message: x
Parts:
- added R18, R19: 2.2K, Resistor_SMD:R_0603_1608Metric, symbol Device:R
- D1, D8: footprint LED_SMD:LED_0603_1608Metric -> dnt:LED_0603_1608Metric - polarity
Connections:
- net GND: now also R18.1
- net at F2.1, L1.2: now also R19.1
- net at U6.3 (FB): now also R18.2, R19.2
Other:
- moved on the sheet: C3, D7, F2

Commit message: 5v buck
Parts:
- added C18, C19: C, Capacitor_SMD:C_0805_2012Metric, symbol Device:C
- added C21: 10uF, Capacitor_SMD:C_0805_2012Metric, symbol Device:C
- added D9: LED-RED, dnt:LED_0603_1608Metric - polarity, symbol Device:LED
- added R21: 2.2K, Resistor_SMD:R_0603_1608Metric, symbol Device:R
- R18: value 2.2K -> 1.02k; LCSC C4190 -> C858881; Manufacturer (none) -> YAGEO; Part # (none) -> RC0603DR-071K02L
- R19: value 2.2K -> 5.62; LCSC C4190 -> C855916; Manufacturer (none) -> YAGEO; Part # (none) -> AT0603BRD075K62L
- U1: footprint dnt:B0505S-1WR2_MNS -> 0505_Isolated_SMD; symbol dnt:B0505S-1WR2 -> dnt:0505_Isolated_SMD; LCSC C C2992393 -> C19188495; MAXIMUM_PACKAGE_HEIGHT (none) -> 6.15mm; Package (none) -> SMD-8 Recom Power; Silkscreen (none) -> XXX
Connections:
- net +3.3V: now also D9.2 (A)
- net +5V: now also C21.1
- net +5V_ISO: now also U1.5 (+VOUT); no longer U1.4 (+VO)
- net GND: now also C19.2, C21.2, R21.1
- net GND_ISO: now also U1.4 (-VOUT); no longer U1.3 (0V)
- net at D7.1 (K), L1.1, U6.6 (SW): now also C18.2
- net at F2.1, L1.2, R19.1: now also C19.1
- net at U6.1 (CB): now also C18.1
- new net: D9.1 (K), R21.2

Commit message: version 2 initial
Parts:
- removed D7: SS14, dnt:D_SMA - polarity, symbol Diode:B340
- added D13: ~, Diode_SMD:D_MicroSMP_AK, symbol Diode:B340
- C4: Manufacturer (none) -> YAGEO; Part Number (none) -> CC0603KRX7R9BB104
Connections:
- net GND: now also D13.2 (A)
- net at C19.1, F2.1, L1.2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: now also C18.2, L1.1, U6.6 (SW), D13.1 (K)
- net at C3.1, D1.2 (A), D2.1 (K)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: now also U6.4 (~{SHDN})

Commit message: version 2 initial- fixes
Parts:
- U100: renamed from U1; value B0505S-1WR2 -> B0505XT-1WR3; footprint 0505_Isolated_SMD -> dnt:0505_Isolated_SMD; Silkscreen XXX -> (none)
Connections:
- net +3.3V renamed +3.3V_REG
Changed lines of the file:
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@@
 			)
 		)
-		(property "Value" "+3.3V"
+		(property "Value" "+3.3V_REG"
 			(at 254 96.52 0)
 			(effects
@@
 		(dnp no)
 		(fields_autoplaced yes)
-		(property "Reference" "U1"
+		(property "Reference" "U100"
 			(at 193.04 133.35 0)
 			(effects
@@
 			)
 		)
-		(property "Value" "B0505S-1WR2"
+		(property "Value" "B0505XT-1WR3"
 			(at 193.04 135.89 0)
 			(effects
@@
 			)
 		)
-		(property "Footprint" "0505_Isolated_SMD"
+		(property "Footprint" "dnt:0505_Isolated_SMD"
 			(at 193.04 146.05 0)
 			(effects
@@
 			)
 		)
-		(property "Description" ""
-			(at 193.04 146.05 0)
-			(effects
-				(font
-					(size 1.27 1.27)
-				)
-				(hide yes)
-			)
-		)
-		(property "Silkscreen" "XXX"
+		(property "Description" "SMD-5 Isolated Power Modules ROHS"
 			(at 193.04 146.05 0)
 			(effects
@@
 			(project "l8-kicad"
 				(path "/8d063f79-9282-4820-bcf4-1ff3c006cf08/cb7fc79f-a21e-4f3e-a003-80932d60a7a0"
-					(reference "U1")
+					(reference "U100")
 					(unit 1)
 				)

Commit message: SENT TO jlcpcb
Parts:
- removed U100: B0505XT-1WR3, dnt:0505_Isolated_SMD, symbol dnt:0505_Isolated_SMD
- added C27, C28: 10uF, Capacitor_SMD:C_0603_1608Metric, symbol Device:C
- added U1: B0505XT-1WR3, dnt:0505_Isolated_SMD, symbol dnt:0505_Isolated_SMD
- C18: value C -> 100nF; footprint Capacitor_SMD:C_0805_2012Metric -> Capacitor_SMD:C_0603_1608Metric; LCSC (none) -> C14663; Manufacturer (none) -> YAGEO; Part Number (none) -> CC0603KRX7R9BB104
- C19: value C -> 22uF; LCSC (none) -> C45783; Voltage (none) -> 25V
- C21: footprint Capacitor_SMD:C_0805_2012Metric -> Capacitor_SMD:C_0603_1608Metric; LCSC C440198 -> C96446; PN GRM21BR61H106KE43L -> (none); Voltage 50V -> (none)
- C3: Vendor (none) -> Murata Electronics
- D1, D8, D9: JLCPCB Rotation Offset 180 -> 0
- D13: value ~ -> MicroSMP(DO-219AD)
- D2: JLCPCB Rotation Offset 180 -> 0; Silkscreen X -> (none)
- R18: value 1.02k -> 10K; LCSC C858881 -> C25804; Manufacturer YAGEO -> StackPole; Part # RC0603DR-071K02L -> RMCF0603JT10K0; VEND (none) -> DIGI; VEND# (none) -> RMCF0603JT10K0CT-ND
- R19: value 5.62 -> 54K9; LCSC C855916 -> C185321; Part # AT0603BRD075K62L -> RC0603FR-0754K9L; Silkscreen (none) -> Hmm
- U6: value LMR14006 -> LMR14006YDDCR; JLCPCB Rotation Offset (none) -> -90; LCSC (none) -> C477919; Order (none) -> https://jlcpcb.com/partdetail/TexasInstruments-LMR14006YDDC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; Package (none) -> TSOT-23-6
Connections:
- net +5V: now also C27.1, U1.2 (+VIN)
- net +5V_ISO: now also C28.1, U1.5 (+VOUT)
- net GND: now also C27.2, U1.1 (-VIN)
- net GND_ISO: now also C28.2, U1.4 (-VOUT)
- net at C18.2, D13.1 (K), L1.1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: no longer C19.1, F2.1, L1.2, R19.1
- net +3.3V_REG renamed +3.3VP
- new net: C19.1, F2.1, L1.2, R19.1
Other:
- note added: "Anode (positive side) and a cathode (negative side)"
- moved on the sheet: C21, C3, C4, C5, C7, D1, D13, D2, D3, D8, D9, F1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

Commit message: update to version 9 on selwyn
Other:
- title: (none) -> l8
